File: eagle/new_object/object_1.brd (EAGLE design)
At the start: 54.6 x 32.8 mm, 13 parts, among them U1 GY-521MPU6050

Commit message: Change switch to pin 23, clean the mess git did with the files
Connections:
- net BTN: now also MS1.23; no longer MS1.22
Routing:
- net BTN: track 22.9 -> 20.3 mm
- net SCL: track 77.5 -> 76.0 mm
Other:
- outline, holes or cut-outs redrawn
Changed lines of the file:
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@@
 <setting verticaltext="up"/>
 </settings>
-<grid distance="0.05" unitdist="inch" unit="mm" style="lines" multiple="1" display="no" altdistance="0.003125" altunitdist="mic" altunit="mm"/>
+<grid distance="0.05" unitdist="inch" unit="mm" style="lines" multiple="1" display="no" altdistance="0.0127" altunitdist="mm" altunit="mm"/>
 <layers>
 <layer number="1" name="Top" color="4" fill="1" visible="yes" active="yes"/>
@@
 <plain>
 <wire x1="60.94" y1="17.018" x2="60.94" y2="44.12" width="0" layer="20"/>
-<wire x1="6.35" y1="44.12" x2="6.35" y2="17.018" width="0" layer="20"/>
+<wire x1="6.35" y1="41.91" x2="6.35" y2="19.05" width="0" layer="20"/>
+<wire x1="6.35" y1="19.05" x2="6.35" y2="17.018" width="0" layer="20"/>
 <wire x1="55.286934375" y1="44.14115" x2="60.937078125" y2="44.13961875" width="0" layer="20" curve="-180"/>
 <wire x1="60.947525" y1="17.00298125" x2="55.29738125" y2="17.0045125" width="0" layer="20" curve="-180"/>
-<wire x1="55.288621875" y1="44.1398" x2="6.35" y2="44.1398" width="0" layer="20"/>
-<wire x1="6.35" y1="44.1398" x2="12.000046875" y2="44.140125" width="0" layer="20"/>
-<wire x1="55.294221875" y1="17.00845" x2="6.35" y2="17.00845" width="0" layer="20"/>
-<wire x1="6.35" y1="17.00845" x2="12.0016375" y2="17.005846875" width="0" layer="20"/>
-<wire x1="12.0016375" y1="17.005846875" x2="12.00495625" y2="17.005846875" width="0" layer="20"/>
+<wire x1="6.35" y1="19.05" x2="14.732" y2="19.05" width="0" layer="20"/>
+<wire x1="55.2958" y1="17.145" x2="55.2958" y2="16.9926" width="0" layer="20"/>
+<wire x1="6.35" y1="41.91" x2="14.732" y2="41.91" width="0" layer="20"/>
+<wire x1="55.2831" y1="43.7515" x2="55.2831" y2="44.1325" width="0" layer="20"/>
+<wire x1="55.2831" y1="43.7515" x2="45.6565" y2="43.7515" width="0" layer="20"/>
+<wire x1="45.6565" y1="43.7515" x2="44.45" y2="42.545" width="0" layer="20"/>
+<wire x1="44.45" y1="42.545" x2="15.367" y2="42.545" width="0" layer="20"/>
+<wire x1="15.367" y1="42.545" x2="14.732" y2="41.91" width="0" layer="20"/>
+<wire x1="55.2958" y1="17.145" x2="52.07" y2="17.145" width="0" layer="20"/>
+<wire x1="52.07" y1="17.145" x2="50.8" y2="18.415" width="0" layer="20"/>
+<wire x1="50.8" y1="18.415" x2="15.367" y2="18.415" width="0" layer="20"/>
+<wire x1="15.367" y1="18.415" x2="14.732" y2="19.05" width="0" layer="20"/>
 </plain>
 <attributes>
@@
 <vertex x="5.08" y="49.53"/>
 </polygon>
+<via x="16.45" y="32.55" extent="1-16" drill="0.8" shape="square"/>
+<via x="18.9" y="32.55" extent="1-16" drill="0.8" shape="square"/>
+<via x="21.7" y="29.05" extent="1-16" drill="0.8" shape="square"/>
+<via x="21.7" y="26.25" extent="1-16" drill="0.8" shape="square"/>
+<wire x1="18.9" y1="32.55" x2="16.45" y2="32.55" width="0" layer="19" extent="1-1"/>
+<wire x1="21.7" y1="26.25" x2="21.7" y2="29.05" width="0" layer="19" extent="1-1"/>
 </signal>
 <signal name="VBAT">
@@
 <wire x1="13.97" y1="27.94" x2="13.97" y2="24.13" width="0.3048" layer="16"/>
 <contactref element="X1" pad="1"/>
-<wire x1="43.18" y1="40.64" x2="43.18" y2="43.18" width="0.4064" layer="16"/>
-<wire x1="43.18" y1="43.18" x2="52.07" y2="43.18" width="0.4064" layer="16"/>
 <wire x1="52.07" y1="43.18" x2="53.34" y2="41.91" width="0.4064" layer="16"/>
 <wire x1="53.34" y1="41.91" x2="54.61" y2="41.91" width="0.4064" layer="16"/>
+<wire x1="52.07" y1="43.18" x2="45.72" y2="43.18" width="0.4064" layer="16"/>
+<wire x1="45.72" y1="43.18" x2="43.18" y2="40.64" width="0.4064" layer="16"/>
 </signal>
 <signal name="SDA">
@@
 </signal>
 <signal name="BTN">
-<contactref element="MS1" pad="22"/>
 <contactref element="JP1" pad="3"/>
-<wire x1="33.02" y1="40.64" x2="33.02" y2="38.1" width="0.4064" layer="16"/>
-<wire x1="33.02" y1="38.1" x2="26.67" y2="38.1" width="0.4064" layer="16"/>
+<wire x1="30.48" y1="38.1" x2="26.67" y2="38.1" width="0.4064" layer="16"/>
 <wire x1="26.67" y1="38.1" x2="26.67" y2="29.21" width="0.4064" layer="16"/>
 <wire x1="26.67" y1="29.21" x2="31.75" y2="29.21" width="0.4064" layer="16"/>
+<contactref element="MS1" pad="23"/>
+<wire x1="30.48" y1="38.1" x2="30.48" y2="40.64" width="0.4064" layer="16"/>
 </signal>
 <signal name="N$2">
